File: kicad-shield-mechanical/kicad-shield-mechanical.kicad_pcb (KiCad board)
At the start: 2 copper layers, 94 x 94 mm, 1258 parts

Commit message: update footprint
Routing:
- net (no net): track 0.00 -> 458.5 mm
