File: kicad-shield-mechanical/kicad-shield-mechanical.kicad_pcb (KiCad board)
At the start: 2 copper layers, 94 x 94 mm, 1258 parts

Commit message: change mounting hole and remove component near cut out
Parts:
- removed 1085, 1086, 1087: , 
- removed the ? at (133.8, 111.0)
- added REF**: MountingHole_3.2mm_6mm_Pad_TopBottom, mykicad_lib:MountingHole_3.2mm_6mm_Pad_TopBottom, F.Cu at (53.5, 53.5)
- added REF**: MountingHole_3.2mm_6mm_Pad_TopBottom, mykicad_lib:MountingHole_3.2mm_6mm_Pad_TopBottom, F.Cu at (140.5, 140.5)
- added REF**: MountingHole_3.2mm_6mm_Pad_TopBottom, mykicad_lib:MountingHole_3.2mm_6mm_Pad_TopBottom, F.Cu at (53.5, 140.5)
- added REF**: MountingHole_3.2mm_6mm_Pad_TopBottom, mykicad_lib:MountingHole_3.2mm_6mm_Pad_TopBottom, F.Cu at (140.5, 53.5)
Routing:
- net (no net): vias 7 -> 0
